File: Single Layer/RAUPS_SingleLayer_Heater.sch (EAGLE design)
At the start: 21 parts, among them Q1 STP55NF06L, Q2 STP55NF06L

Commit message: Added BOM, final single layer board tweaks, and re-organized file structure to better reflect project goals
Parts:
- C6: value 470uF -> 100uF
Changed lines of the file:
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@@
 <part name="R9" library="adafruit" deviceset="R-US_" device="0207/7" value="100k"/>
 <part name="C4" library="capacitor-wima" deviceset="C" device="2,5-3" value="100nF"/>
-<part name="C6" library="adafruit" deviceset="CPOL-US" device="E3.5-8" value="470uF"/>
+<part name="C6" library="adafruit" deviceset="CPOL-US" device="E3.5-8" value="100uF"/>
 <part name="F1" library="RepRapjr" deviceset="PTCFUSE" device="" value="MFR500"/>
 <part name="F2" library="RepRapjr" deviceset="PTCFUSE" device="MFR1100" value="MFR1100"/>
